File: PC1500-Pico2W-Dongle-no-level-shifters/PC1500-Pico2W-Dongle.kicad_sch (KiCad schematic)
At the start: 65 parts, among them J1 PC1500_60Pin_Connector, J2 microSD, J3 Spare GPIO (GP28), J5 GP2_Spare_IO, Q1 Si2333, Q2 MMBT2222A, U1 Pico2W, U2 AS6C62256-55SIN, U3 SLG46826G, U4 SLG46826G, U5 SC18IS602B, U6 TXS0108EPWR, U7 AP1117-ADJ, U8 TCA9406DC

Commit message: Pico2W-Dongle-no-level-shifters: I2C pull-ups, cap fixes, SDA1/SCL1 rename, hand-routing
Schematic: R11-R14 I2C pull-up resistors (2K on VGG for SDA_GP/SCL_GP,
1.5K on 3V3 for SDA/SCL), C1/C2/C6/C7/C8 capacitor connections fixed
(were fully or partially unwired), JP1/JP2 renamed to SDA1/SCL1 to
match user's PCB-side silkscreen relabeling.

PCB: C1/C2/C6 net assignments patched to match; SDA1/SCL1 footprint
references renamed to match; user's manual routing/silkscreen fixes.

Known state: 0 unconnected nets, but 100 DRC violations remain (mostly
track_width squeeze escaping fine-pitch GreenPAK/SD-bridge pins, plus
some clearance/silk) -- not yet fab-clean, captured here as a checkpoint.
Parts:
- removed R15, R17, R19, R21, R23, R25, R27, R29, R31, R33, R35, R37, R39: 10k, Resistor_SMD:R_0201_0603Metric, symbol Device:R
- removed R16, R18, R20, R22, R24, R26, R28, R30, R32, R34, R36, R38: 4.7k, Resistor_SMD:R_0201_0603Metric, symbol Device:R
- removed U6: TXS0108EPWR, Package_SO:TSSOP-20_4.4x6.5mm_P0.65mm, symbol Logic_LevelTranslator:TXS0108EPW
- JP3: renamed from Jumper1; value Jumper_2_Bridged -> 1500A; footprint Jumper:SolderJumper-2_P1.3mm_Bridged_RoundedPad1.0x1.5mm -> Connector_PinHeader_2.54mm:PinHeader_1x02_P2.54mm_Vertical; symbol Jumper:Jumper_2_Bridged -> Connector_Generic:Conn_01x02
- R10: value 4.7k -> 10k
- R11: value 10k -> 2K
- R12: value 4.7k -> 2K
- R13: value 10k -> 1.5K
- R14: value 4.7k -> 1.5K
- renumbered JP2 to SCL1, JP1 to SDA1
Connections:
- net AD10_PICO is gone; now on net AD10: U1.14 (GP10)
- net AD11_PICO is gone; now on net AD11: U1.15 (GP11)
- net AD12_PICO is gone; now on net AD12: U1.16 (GP12)
- net AD3_PICO is gone; now on net AD3: U1.5 (GP3)
- net AD4_PICO is gone; now on net AD4: U1.6 (GP4)
- net AD5_PICO is gone; now on net AD5: U1.7 (GP5)
- net AD6_PICO is gone; now on net AD6: U1.9 (GP6)
- net AD7_PICO is gone; now on net AD7: U1.10 (GP7)
- net AD8_PICO is gone; now on net AD8: U1.11 (GP8)
- net AD9_PICO is gone; now on net AD9: U1.12 (GP9)
- net D0_LV is gone; now on net D0: U1.17 (GP13)
- net D1_LV is gone; now on net D1: U1.19 (GP14)
- net D2_LV is gone; now on net D2: U1.20 (GP15)
- net D3_LV is gone; now on net D3: U1.21 (GP16)
- net D4_LV is gone; now on net D4: U1.22 (GP17)
- net D5_LV is gone; now on net D5: U1.24 (GP18)
- net D6_LV is gone; now on net D6: U1.25 (GP19)
- net D7_LV is gone; now on net D7: U1.26 (GP20)
- net TRIG_RD_PICO is gone; now on net TRIG_RD: U1.27 (GP21)
- net TRIG_WR_PICO is gone; now on net TRIG_WR: U1.29 (GP22)
- net +BATT: now also C1.1
- net 3V3: now also C6.1, C8.1, R10.2, R13.1, R14.1
- net AD0: now also U1.1 (GP0); no longer R10.1
- net AD1: now also U1.2 (GP1); no longer R12.1
- net AD2: now also U1.4 (GP2); no longer R14.1
- net GND: now also C1.2, C2.2, C6.2, C7.2, C8.2; no longer J2.3 (VSS), J2.6 (VSS), R11.2, R13.2
- net SCL: now also R14.2
- net SCL_GP: now also R12.2
- net SDA: now also R13.2
- net SDA_GP: now also R11.2
- net SD_CS: now also J2.2 (CMD); no longer J2.1 (CD/DAT3)
- net SD_MOSI: now also J2.3 (VSS), J2.6 (VSS); no longer J2.2 (CMD)
- net VGG: now also C2.1, R11.1, R12.1
- removed net AD0_PICO: R10.2, R11.1, U1.1 (GP0)
- removed net AD1_PICO: R12.2, R13.1, U1.2 (GP1)
- removed net AD2_PICO: R14.2, U1.4 (GP2)
- new net: J2.1 (CD/DAT3), R10.1
Other:
- moved on the sheet: C2, C7, C8, J5
