File: PC1500-Pico2W-Dongle-no-level-shifters/PC1500-Pico2W-Dongle.kicad_pcb (KiCad board)
At the start: 4 copper layers, 61 x 78 mm, 39 parts, among them J1 PC1500_60Pin_Connector, J2 microSD, J3 Spare GPIO (GP28), J5 GP2_Spare_IO, Q1 Si2333, Q2 MMBT2222A, U1 Pico2W, U2 AS6C62256-55SIN, U3 SLG46826G, U4 SLG46826G, U5 SC18IS602B, U7 AP1117-ADJ, U8 TCA9406DC

Commit message: Fix J2 pin 6->GND copper on Pico2W-Dongle-no-level-shifters, export fab files
Pad 6 was still physically bridged in copper to pad 3 (SD_MOSI) despite
the earlier schematic fix; user reworked the PCB to route it to GND
directly. Also re-grounded the 4 shield pads, which lost their GND net
assignment again during the schematic sync (recurring issue since they
have no corresponding schematic pin).

Regenerated Gerbers (Protel extensions + job file), drill files, BOM,
and component placement file for this board. The CPL was rebuilt with
JLCPCB's expected header (Designator,Mid X,Mid Y,Layer,Rotation instead
of KiCad's default Ref,Val,Package,PosX,PosY,Rot,Side) and normalized
rotations to 0-360 degrees, since JLCPCB's uploader could not read the
previous file.

Co-Authored-By: Claude Sonnet 5 <noreply@anthropic.com>
Parts:
- J3: value Spare GPIO (GP28) -> INT / GP28 / GND; footprint Connector_PinHeader_2.54mm:PinHeader_1x02_P2.54mm_Vertical -> Connector_PinHeader_2.54mm:PinHeader_1x03_P2.54mm_Vertical
- moved J3 2.54 mm to (53.5, 9.46)
Connections:
- J2 pad 6: SD_MOSI -> GND
- J2 pad SH: (no net) -> GND
- J3 pad 1: GP28 -> ~INT
- J3 pad 2: GND -> GP28
- U5 pad 9: unconnected-(U5-~INT-Pad9) -> ~INT
Routing:
- net ~INT: track 0.00 -> 9.80 mm
- net SD_MOSI: track 55.9 -> 51.1 mm
- net GND: track 33.2 -> 33.6 mm, vias 13 -> 17
Changed lines of the file:
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@@
 		)
 	)
-	(footprint "Connector_PinHeader_2.54mm:PinHeader_1x02_P2.54mm_Vertical"
+	(footprint "Connector_PinHeader_2.54mm:PinHeader_1x03_P2.54mm_Vertical"
 		(layer "F.Cu")
-		(at 53.5 12)
-		(descr "Through hole straight pin header, 1x02, 2.54mm pitch, single row")
-		(tags "Through hole pin header THT 1x02 2.54mm single row")
+		(at 53.5 9.46)
+		(descr "Through hole straight pin header, 1x03, 2.54mm pitch, single row")
+		(tags "Through hole pin header THT 1x03 2.54mm single row")
 		(property "Reference" "J3"
 			(at 0 -2.38 0)
@@
 			)
 		)
-		(property "Value" "Spare GPIO (GP28)"
-			(at 0 4.92 0)
+		(property "Value" "INT / GP28 / GND"
+			(at 0 7.46 0)
 			(layer "F.Fab")
 			(effects
@@
 			)
 		)
-		(property ki_fp_filters "Connector*:*_1x??_*")
 		(sheetname "/")
 		(sheetfile "PC1500-Pico2W-Dongle.kicad_sch")
@@
 			(unit
 				(name "A")
-				(pins "1" "2")
+				(pins "1" "2" "3")
 			)
 		)
@@
 		(fp_line
 			(start -1.38 1.27)
-			(end -1.38 3.92)
+			(end -1.38 6.46)
 			(stroke
 				(width 0.12)
@@
 		)
 		(fp_line
-			(start -1.38 3.92)
-			(end 1.38 3.92)
+			(start -1.38 6.46)
+			(end 1.38 6.46)
 			(stroke
 				(width 0.12)
@@
 		(fp_line
 			(start 1.38 1.27)
-			(end 1.38 3.92)
+			(end 1.38 6.46)
 			(stroke
 				(width 0.12)
@@
 		(fp_rect
 			(start -1.77 -1.77)
-			(end 1.77 4.32)
+			(end 1.77 6.85)
 			(stroke
 				(width 0.05)
@@
 		)
 		(fp_line
-			(start -1.27 3.81)
+			(start -1.27 6.35)
 			(end -1.27 -0.635)
 			(stroke
@@
 		(fp_line
 			(start 1.27 -1.27)
-			(end 1.27 3.81)
+			(end 1.27 6.35)
 			(stroke
 				(width 0.1)
@@
 		)
 		(fp_line
-			(start 1.27 3.81)
-			(end -1.27 3.81)
+			(start 1.27 6.35)
+			(end -1.27 6.35)
 			(stroke
 				(width 0.1)
@@
 			(layer "F.Fab")
 		)
+		(fp_text user "INT"
+			(at 1.2 0 0)
+			(layer "F.SilkS")
+			(effects
+				(font
+					(size 0.8 0.8)
+					(thickness 0.12)
+				)
+				(justify left)
+			)
+		)
+		(fp_text user "GP28"
+			(at 1.2 2.54 0)
+			(layer "F.SilkS")
+			(effects
+				(font
+					(size 0.8 0.8)
+					(thickness 0.12)
+				)
+				(justify left)
+			)
+		)
+		(fp_text user "GND"
+			(at 1.2 5.08 0)
+			(layer "F.SilkS")
+			(effects
+				(font
+					(size 0.8 0.8)
+					(thickness 0.12)
+				)
+				(justify left)
+			)
+		)
 		(fp_text user "${REFERENCE}"
-			(at 0 1.27 90)
+			(at 0 2.54 90)
 			(layer "F.Fab")
 			(effects
@@
 			(layers "*.Cu" "*.Mask")
 			(remove_unused_layers no)
-			(net "GP28")
+			(net "~INT")
 			(pinfunction "Pin_1_1")
 			(pintype "passive")
@@
 			(layers "*.Cu" "*.Mask")
 			(remove_unused_layers no)
-			(net "GND")
+			(net "GP28")
 			(pinfunction "Pin_2_2")
 			(pintype "passive")
 		)
+		(pad "3" thru_hole circle
+			(at 0 5.08)
+			(size 1.7 1.7)
+			(drill 1)
+			(layers "*.Cu" "*.Mask")
+			(remove_unused_layers no)
+			(net "GND")
+			(pinfunction "Pin_3_3")
+			(pintype "passive")
+		)
 		(embedded_fonts no)
-		(model "${KICAD10_3DMODEL_DIR}/Connector_PinHeader_2.54mm.3dshapes/PinHeader_1x02_P2.54mm_Vertical.step"
+		(model "${KICAD10_3DMODEL_DIR}/Connector_PinHeader_2.54mm.3dshapes/PinHeader_1x03_P2.54mm_Vertical.step"
 			(offset
 				(xyz 0 0 0)
@@
 			(size 0.85 1.1)
 			(layers "F.Cu" "F.Mask" "F.Paste")
-			(net "SD_MOSI")
+			(net "GND")
 			(pinfunction "VSS_6")
 			(pintype "passive")
@@
 			(size 1.55 1.35)
 			(layers "F.Cu" "F.Mask" "F.Paste")
+			(net "GND")
 		)
 		(pad "SH" smd rect
@@
 			(size 1.9 1.35)
 			(layers "F.Cu" "F.Mask" "F.Paste")
+			(net "GND")
 		)
 		(pad "SH" smd rect
@@
 			(size 1.9 1.35)
 			(layers "F.Cu" "F.Mask" "F.Paste")
+			(net "GND")
 		)
 		(pad "SH" smd rect
@@
 			(size 1.17 1.8)
 			(layers "F.Cu" "F.Mask" "F.Paste")
+			(net "GND")
 		)
 		(embedded_fonts no)
@@
 			(layers "F.Cu" "F.Mask" "F.Paste")
 			(roundrect_rratio 0.25)
-			(net "unconnected-(U5-~INT-Pad9)")
+			(net "~INT")
 			(pinfunction "~INT_9")
 			(pintype "output")
@@
 	)
 	(segment
+		(start 11.395 3.0746)
+		(end 11.395 3.55)
+		(width 0.2)
+		(layer "F.Cu")
+		(net "GND")
+	)
+	(segment
 		(start 46.8 19.2)
 		(end 46.775 19.2)
@@
 	)
 	(via
+		(at 11.395 3.3677)
+		(size 0.6)
+		(drill 0.3)
+		(layers "F.Cu" "B.Cu")
+		(net "GND")
+	)
+	(via
 		(at 31.625 20)
 		(size 0.6)
@@
 	)
 	(via
+		(at 5.9 14.375)
+		(size 0.6)
+		(drill 0.3)
+		(layers "F.Cu" "B.Cu")
+		(net "GND")
+	)
+	(via
+		(at 3.435 3.675)
+		(size 0.6)
+		(drill 0.3)
+		(layers "F.Cu" "B.Cu")
+		(net "GND")
+	)
+	(via
 		(at 18 61.6)
 		(size 0.6)
@@
 	)
 	(via
+		(at 12.73 14.375)
+		(size 0.6)
+		(drill 0.3)
+		(layers "F.Cu" "B.Cu")
+		(net "GND")
+	)
+	(via
 		(at 43.2 8.4)
 		(size 0.6)
@@
 	)
 	(segment
+		(start 50.685 12.275)
+		(end 44.8625 12.275)
+		(width 0.2)
+		(layer "F.Cu")
+		(net "~INT")
+	)
+	(segment
+		(start 53.5 9.46)
+		(end 50.685 12.275)
+		(width 0.2)
+		(layer "F.Cu")
+		(net "~INT")
+	)
+	(segment
 		(start 38.9678 29.825)
 		(end 40.4214 28.3714)
@@
 	)
 	(segment
-		(start 11.0202 2.6998)
-		(end 11.395 3.0746)
-		(width 0.2)
-		(layer "F.Cu")
-		(net "SD_MOSI")
-	)
-	(segment
-		(start 8.095 3.55)
-		(end 8.095 2.6998)
-		(width 0.2)
-		(layer "F.Cu")
-		(net "SD_MOSI")
-	)
-	(segment
 		(start 8.095 4.6045)
 		(end 8.095 3.55)
@@
 		(layer "F.Cu")
 		(net "SD_MOSI")
-	)
-	(segment
-		(start 11.395 3.0746)
-		(end 11.395 3.55)
-		(width 0.2)
-		(layer "F.Cu")
-		(net "SD_MOSI")
-	)
-	(segment
-		(start 8.095 2.6998)
-		(end 11.0202 2.6998)
-		(width 0.15)
-		(layer "F.Cu")
-		(net "SD_MOSI")

Commit message: Pico 2 W dongle (no level shifters): current schematic and PCB
The board owner's schematic and PCB as saved 2026-10-03/04.

Co-Authored-By: Claude Opus 5.5 <noreply@anthropic.com>
Parts:
- added R15: 4.7k, Resistor_SMD:R_0201_0603Metric, F.Cu at (50.0, 15.4)
- J1: value PC1500_60Pin_Connector -> PC1500 60Pin Connector
- J5: value GP2_Spare_IO -> GP2 Spare IO
- Q1, Q2, R3, R4: moved to F.Cu
- R1, R2: footprint Resistor_SMD:R_0201_0603Metric -> Resistor_SMD:R_0603_1608Metric
- SCL1, SDA1: value GP1-GP2 I2C link -> GP1 GP2 I2C link
- U2: value AS6C62256-55SIN -> AS6C62256 55SIN
- U7: value AP1117-ADJ -> NCP1117 ADJ
- moved R4 64.4 mm to (50.0, 17.0), turned to 90 degrees
- moved Q1 59.4 mm to (40.8, 18.0)
- moved R3 58.6 mm to (43.4, 18.0), turned to -90 degrees
- moved Q2 58.3 mm to (47.4, 15.4)
- moved C4 9.77 mm to (21.2, 61.0), turned to -90 degrees
- moved R2 2.50 mm to (40.0, 37.2)
- moved R1 1.88 mm to (40.6, 34.8), turned to 180 degrees
Connections:
- net +4V7 renamed VCC
- J1 pad 15: PV -> PU
- J1 pad 16: PU -> PV
- J2 pad SH: GND -> (no net)
- Q1 pad 1: (no net) -> Net-(Q1-G)
- Q1 pad 2: (no net) -> VGG
- Q1 pad 3: (no net) -> VSYS_SW
- Q2 pad 1: (no net) -> Net-(Q2-B)
- Q2 pad 2: (no net) -> GND
- Q2 pad 3: (no net) -> Net-(Q1-G)
- R3 pad 2: GATE_NODE -> Net-(Q1-G)
- R4 pad 2: Q2_BASE -> Net-(Q2-B)
Routing:
- net VGG: track 141.1 -> 121.6 mm
- net VCC: track 63.5 -> 47.3 mm
- net Net-(Q1-G): track 0.00 -> 8.12 mm, vias 0 -> 2
- net VGG_FB: track 25.5 -> 18.9 mm
- net VSYS_SW: track 0.00 -> 6.13 mm
- net PV: track 44.1 -> 47.4 mm
- net Net-(Q2-B): track 0.00 -> 2.68 mm
- net GP28: track 29.4 -> 30.2 mm
- net SD_MOSI: vias 2 -> 3
