File: PC1500-RP2350B-BLE/PC1500-RP2350B-BLE.kicad_pcb (KiCad board)
At the start: 8 copper layers, 31.9 x 43 mm, 44 parts, among them J1 microSD, J2 USB-C (programming/debug), J3 PC-1500 40-pin cartridge slot, J5 PC1500_SENSE_JUMPER, J6 SPARE_GPIO_U9, J7 SWD_I2C_HEADER, SW1 BOOTSEL, U1 RP2350B, U10 TCA9406DCUR, U11 FXMA108, U12 FXMA108, U2 AS6C62256-55STCN, U3 SLG46826V, U4 AP2112K-3.3, U5 W25Q32RVXHJQ, U7 FXMA108, U8 RN4871, U9 SLG46826V, X1 12MHz (Abracon ABM8-272-T3)

Commit message: Boards: card-edge pinout and X1 fixes; More-RAM, ROM replacement, adapter
- Card edge (J3), all boards: viewed from the top with the edge up,
  pin 1 is on the right, 21 under 1, 40 under 20. The pads were mirrored;
  fixed in place, no rerouting.
- X1 (ABM8): the 4-pad crystal had the 2-pin Device:Crystal symbol. Now
  Device:Crystal_GND24 (XIN 1, XOUT 3, GND 2/4) on More-RAM and both
  RP2350B-BLE boards.
- PC1500-RP2354B-BLE-more-RAM (the internal card), new in git:
  - BGM220SC22WGA2 replaces the RN4871: footprint from datasheet Rev 1.4
    with the antenna loop on ANT_OUT, no copper under the antenna or its
    keepout, a ground pour around the module only, thermal-relief centre
    pads; R24 0R between ANT_IN and RF_2G4.
  - D0-D7 on GPIO16-23 in order (the PIO window); GREENPAK2_IO14 on
    GPIO25 (5 V tolerant); UART0 GPIO32-35, RESETn 36, HOST_WAKE 37,
    SWD 38/39, BLE_MODULE_WAKE GPIO27 -> PB03.
  - SD_MISO reconnected to GPIO40 (a label 1.27 mm off the pin end).
  - Signal netclass for every signal net.
- PC1500-ROM-Replacement-Board and PC-1500-40-pin-Breadboard-Adapter
  (Sullins RBB20DHHN socket, DIP-40 and DIP-28 hole rows), new in git.
- .gitignore: scripted-edit backups, KiCad history and editor locks.

Design files only: fab/production outputs aren't included (More-RAM's
fab/ predates these changes).

Co-Authored-By: Claude Opus 5.5 <noreply@anthropic.com>
Connections:
- X1 pad 2: XOUT -> GND
- X1 pad 3: (no net) -> XOUT
- X1 pad 4: (no net) -> GND
