File: PC1500-RP2350B-BLE/PC1500-RP2350B-BLE.kicad_sch (KiCad schematic)
At the start: 44 parts, among them J1 microSD, J2 USB-C (programming/debug), J3 PC-1500 40-pin cartridge slot, J5 PC1500_SENSE_JUMPER, J6 SPARE_GPIO_U9, J7 SWD_I2C_HEADER, SW1 BOOTSEL, U1 RP2350B, U10 TCA9406DCUR, U11 FXMA108, U12 FXMA108, U2 AS6C62256-55STCN, U3 SLG46826V, U4 AP2112K-3.3, U5 W25Q32RVXHJQ, U7 FXMA108, U8 RN4871, U9 SLG46826V, X1 12MHz (Abracon ABM8-272-T3)

Commit message: Fix microSD pin 6 (GND) and pin 1 (unused, needs pull-up) on all 4 boards
Pin 6 and pin 3 were coincident in the generic SD_Card_Device symbol,
forcing GND onto the same net as CMD/MOSI. Relocated pin 6's local
coordinate and gave it its own wire+label on all four schematics
(RP2350B-BLE and Pico2W-Dongle, each with and without level shifters).

Pin 1 (symbol name CD/DAT3) is unused in this design but needs a 10K
pull-up to 3.3V rather than being left floating, matching the existing
SD_CS/SD_MOSI/SD_DAT1/SD_DAT2 pull-up pattern. Added the missing
wire+label+resistor to the three boards that lacked it
(Pico2W-Dongle-no-level-shifters already had it via R10).

Co-Authored-By: Claude Sonnet 5 <noreply@anthropic.com>
Parts:
- added R19: 10K, Resistor_SMD:R_0201_0603Metric, symbol Device:R
Connections:
- net +3V3: now also R19.1
- net GND: no longer J1.3 (VSS)
- net SD_CS: now also J1.2 (CMD); no longer J1.1 (CD/DAT3)
- net SD_MOSI: now also J1.3 (VSS); no longer J1.2 (CMD)
- new net CD_DAT3: J1.1 (CD/DAT3), R19.2
Changed lines of the file:
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@@
 	(wire
 		(pts
-			(xy 264.76 227.46) (xy 267.3 227.46)
-		)
-		(stroke
-			(width 0)
-			(type default)
-		)
-	)
-	(wire
-		(pts
 			(xy 397.56 243.84) (xy 396.24 243.84)
 		)
@@
 	(wire
 		(pts
+			(xy 282.54 247.78) (xy 285.08 247.78)
+		)
+		(stroke
+			(width 0)
+			(type default)
+		)
+		(uuid "j1gnd0001-a1a1-4000-8000-j1gnd00001")
+	)
+	(global_label "GND"
+		(shape input)
+		(at 285.08 247.78 0)
+		(effects
+			(font
+				(size 1.27 1.27)
+			)
+			(justify left)
+		)
+		(uuid "j1gnd0002-a1a1-4000-8000-j1gnd00002")
+		(property "Intersheetrefs" "${INTERSHEET_REFS}"
+			(at 285.08 247.78 0)
+			(hide yes)
+			(show_name no)
+			(do_not_autoplace no)
+			(effects
+				(font
+					(size 1.27 1.27)
+				)
+			)
+		)
+	)
+	(wire
+		(pts
 			(xy 325 132.38) (xy 325 129.84)
 		)
@@
 		)
 	)
-	(global_label "SD_MOSI"
+	(global_label "SD_CS"
 		(shape input)
 		(at 267.3 235.08 0)
@@
 		)
 	)
+	(wire
+		(pts
+			(xy 264.76 227.46) (xy 267.3 227.46)
+		)
+		(stroke
+			(width 0)
+			(type default)
+		)
+		(uuid "j1pu10001-a1a1-4000-8000-j1pu1000001")
+	)
+	(global_label "CD_DAT3"
+		(shape input)
+		(at 267.3 227.46 0)
+		(effects
+			(font
+				(size 1.27 1.27)
+			)
+			(justify left)
+		)
+		(uuid "j1pu10002-a1a1-4000-8000-j1pu1000002")
+		(property "Intersheetrefs" "${INTERSHEET_REFS}"
+			(at 267.3 227.46 0)
+			(hide yes)
+			(show_name no)
+			(do_not_autoplace no)
+			(effects
+				(font
+					(size 1.27 1.27)
+				)
+			)
+		)
+	)
+	(wire
+		(pts
+			(xy 324 193.81) (xy 324 196.35)
+		)
+		(stroke
+			(width 0)
+			(type default)
+		)
+		(uuid "j1pu10003-a1a1-4000-8000-j1pu1000003")
+	)
+	(global_label "CD_DAT3"
+		(shape input)
+		(at 324 196.35 0)
+		(effects
+			(font
+				(size 1.27 1.27)
+			)
+			(justify left)
+		)
+		(uuid "j1pu10004-a1a1-4000-8000-j1pu1000004")
+		(property "Intersheetrefs" "${INTERSHEET_REFS}"
+			(at 324 196.35 0)
+			(hide yes)
+			(show_name no)
+			(do_not_autoplace no)
+			(effects
+				(font
+					(size 1.27 1.27)
+				)
+			)
+		)
+	)
+	(wire
+		(pts
+			(xy 324 186.19) (xy 324 183.65)
+		)
+		(stroke
+			(width 0)
+			(type default)
+		)
+		(uuid "j1pu10005-a1a1-4000-8000-j1pu1000005")
+	)
+	(global_label "+3V3"
+		(shape input)
+		(at 324 183.65 0)
+		(effects
+			(font
+				(size 1.27 1.27)
+			)
+			(justify left)
+		)
+		(uuid "j1pu10006-a1a1-4000-8000-j1pu1000006")
+		(property "Intersheetrefs" "${INTERSHEET_REFS}"
+			(at 324 183.65 0)
+			(hide yes)
+			(show_name no)
+			(do_not_autoplace no)
+			(effects
+				(font
+					(size 1.27 1.27)
+				)
+			)
+		)
+	)
 	(global_label "CC2_R"
 		(shape input)
@@
 		)
 	)
-	(global_label "GND"
+	(global_label "SD_MOSI"
 		(shape input)
 		(at 280 245.24 0)
@@
 		)
 	)
-	(global_label "SD_CS"
-		(shape input)
-		(at 267.3 227.46 0)
-		(effects
-			(font
-				(size 1.27 1.27)
-			)
-			(justify left)
-		)
-		(property "Intersheetrefs" "${INTERSHEET_REFS}"
-			(at 267.3 227.46 0)
-			(hide yes)
-			(show_name no)
-			(do_not_autoplace no)
-			(effects
-				(font
-					(size 1.27 1.27)
-				)
-			)
-		)
-	)
 	(global_label "SD_MISO"
 		(shape input)
@@
 					(unit 1)
 				)
+			)
+		)
+	)
+	(symbol
+		(lib_id "Device:R")
+		(at 324 190 0)
+		(unit 1)
+		(body_style 1)
+		(exclude_from_sim no)
+		(in_bom yes)
+		(on_board yes)
+		(in_pos_files yes)
+		(dnp no)
+		(uuid "j1pu1r19-a1a1-4000-8000-j1pu1r19001")
+		(property "Reference" "R19"
+			(at 324 185 0)
+			(show_name no)
+			(do_not_autoplace no)
+			(effects
+				(font
+					(size 1.27 1.27)
+				)
+			)
+		)
+		(property "Value" "10K"
+			(at 324 195 0)
+			(show_name no)
+			(do_not_autoplace no)
+			(effects
+				(font
+					(size 1.27 1.27)
+				)
+			)
+		)
+		(property "Footprint" "Resistor_SMD:R_0201_0603Metric"
+			(at 324 190 0)
+			(hide yes)
+			(show_name no)
+			(do_not_autoplace no)
+			(effects
+				(font
+					(size 1.27 1.27)
+				)
+			)
+		)
+		(property "Datasheet" ""
+			(at 324 190 0)
+			(show_name no)
+			(do_not_autoplace no)
+			(effects
+				(font
+					(size 1.27 1.27)
+				)
+			)
+		)
+		(property "Description" ""
+			(at 324 190 0)
+			(show_name no)
+			(do_not_autoplace no)
+			(effects
+				(font
+					(size 1.27 1.27)
+				)
+			)
+		)
+		(pin "1"
+			(uuid "j1pu1r19-a1a1-4000-8000-j1pu1r19002")
+		)
+		(pin "2"
+			(uuid "j1pu1r19-a1a1-4000-8000-j1pu1r19003")
+		)
+		(instances
+			(project "PC1500-RP2350B-BLE"
+				(path "/3452a646-cdf9-46e9-9c5b-7a6b57374bfc"
+					(reference "R19")
+					(unit 1)
+				)

Commit message: Boards: card-edge pinout and X1 fixes; More-RAM, ROM replacement, adapter
- Card edge (J3), all boards: viewed from the top with the edge up,
  pin 1 is on the right, 21 under 1, 40 under 20. The pads were mirrored;
  fixed in place, no rerouting.
- X1 (ABM8): the 4-pad crystal had the 2-pin Device:Crystal symbol. Now
  Device:Crystal_GND24 (XIN 1, XOUT 3, GND 2/4) on More-RAM and both
  RP2350B-BLE boards.
- PC1500-RP2354B-BLE-more-RAM (the internal card), new in git:
  - BGM220SC22WGA2 replaces the RN4871: footprint from datasheet Rev 1.4
    with the antenna loop on ANT_OUT, no copper under the antenna or its
    keepout, a ground pour around the module only, thermal-relief centre
    pads; R24 0R between ANT_IN and RF_2G4.
  - D0-D7 on GPIO16-23 in order (the PIO window); GREENPAK2_IO14 on
    GPIO25 (5 V tolerant); UART0 GPIO32-35, RESETn 36, HOST_WAKE 37,
    SWD 38/39, BLE_MODULE_WAKE GPIO27 -> PB03.
  - SD_MISO reconnected to GPIO40 (a label 1.27 mm off the pin end).
  - Signal netclass for every signal net.
- PC1500-ROM-Replacement-Board and PC-1500-40-pin-Breadboard-Adapter
  (Sullins RBB20DHHN socket, DIP-40 and DIP-28 hole rows), new in git.
- .gitignore: scripted-edit backups, KiCad history and editor locks.

Design files only: fab/production outputs aren't included (More-RAM's
fab/ predates these changes).

Co-Authored-By: Claude Opus 5.5 <noreply@anthropic.com>
Parts:
- X1: symbol Device:Crystal -> Device:Crystal_GND24
Connections:
- net GND: now also X1.2 (G), X1.4 (G)
- net XOUT: now also X1.3; no longer X1.2
Changed lines of the file:
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@@
 	)
 	(symbol
-		(lib_id "Device:Crystal")
+		(lib_id "Device:Crystal_GND24")
 		(at 340 140 0)
 		(unit 1)
@@
 		)
 		(property "Value" "12MHz (Abracon ABM8-272-T3)"
-			(at 340 145 0)
+			(at 340 151.43 0)
 			(show_name no)
 			(do_not_autoplace no)
@@
 		)
 		(pin "2"
+		)
+		(pin "3"
+		)
+		(pin "4"
 		)
 		(instances
@@
 			(hide yes)
 			(show_name no)
+			(do_not_autoplace no)
+			(effects
+				(font
+					(size 1.27 1.27)
+				)
+			)
+		)
+	)
+	(wire
+		(pts
+			(xy 340 145.08) (xy 340 147.62)
+		)
+		(stroke
+			(width 0)
+			(type default)
+		)
+	)
+	(global_label "GND"
+		(shape bidirectional)
+		(at 340 147.62 0)
+		(effects
+			(font
+				(size 1.27 1.27)
+			)
+			(justify left)
+		)
+		(property "Intersheetrefs" "${INTERSHEET_REFS}"
+			(at 340 147.62 0)
+			(hide yes)
+			(show_name no)
