File: PC1500-RP2350B-BLE-no-level-shifters/PC1500-RP2350B-BLE.kicad_pcb (KiCad board)
At the start: 8 copper layers, 31.9 x 43 mm, 40 parts, among them J1 microSD, J2 USB-C (programming/debug), J3 PC-1500 40-pin cartridge slot, J5 PC1500_SENSE_JUMPER, J6 SPARE_GPIO_U9, J7 SWD_I2C_HEADER, SW1 BOOTSEL, U1 RP2354B, U10 TCA9406DCUR, U2 AS6C62256-55STCN, U3 SLG46826V, U4 AP2112K-3.3, U8 RN4871, U9 SLG46826V, X1 12MHz (Abracon ABM8-272-T3)

Commit message: Boards: card-edge pinout and X1 fixes; More-RAM, ROM replacement, adapter
- Card edge (J3), all boards: viewed from the top with the edge up,
  pin 1 is on the right, 21 under 1, 40 under 20. The pads were mirrored;
  fixed in place, no rerouting.
- X1 (ABM8): the 4-pad crystal had the 2-pin Device:Crystal symbol. Now
  Device:Crystal_GND24 (XIN 1, XOUT 3, GND 2/4) on More-RAM and both
  RP2350B-BLE boards.
- PC1500-RP2354B-BLE-more-RAM (the internal card), new in git:
  - BGM220SC22WGA2 replaces the RN4871: footprint from datasheet Rev 1.4
    with the antenna loop on ANT_OUT, no copper under the antenna or its
    keepout, a ground pour around the module only, thermal-relief centre
    pads; R24 0R between ANT_IN and RF_2G4.
  - D0-D7 on GPIO16-23 in order (the PIO window); GREENPAK2_IO14 on
    GPIO25 (5 V tolerant); UART0 GPIO32-35, RESETn 36, HOST_WAKE 37,
    SWD 38/39, BLE_MODULE_WAKE GPIO27 -> PB03.
  - SD_MISO reconnected to GPIO40 (a label 1.27 mm off the pin end).
  - Signal netclass for every signal net.
- PC1500-ROM-Replacement-Board and PC-1500-40-pin-Breadboard-Adapter
  (Sullins RBB20DHHN socket, DIP-40 and DIP-28 hole rows), new in git.
- .gitignore: scripted-edit backups, KiCad history and editor locks.

Design files only: fab/production outputs aren't included (More-RAM's
fab/ predates these changes).

Co-Authored-By: Claude Opus 5.5 <noreply@anthropic.com>
Parts:
- added R19: 10K, Resistor_SMD:R_0201_0603Metric, B.Cu at (163.2, 89.8)
Connections:
- net GREENPAK1_SCL renamed SCL
- net GREENPAK1_SDA renamed SDA
- J1 pad 1: SD_CS -> CD_DAT3
- J1 pad 2: SD_MOSI -> SD_CS
- J1 pad 3: GND -> SD_MOSI
- TP1 pad 1: Net-(U9-IO6) -> TRIG_RD
- TP3 pad 1: Net-(U9-IO4) -> AD15
- U2 pad 17: unconnected-(U2-Q5-Pad17) -> D5
- U3 pad 1: DME0 -> VGG
- U3 pad 10: GND -> SRAM_A11
- U3 pad 11: unconnected-(U3-IO6-Pad11) -> GND
- U3 pad 12: SDA_GP -> SRAM_A12
- U3 pad 13: SCL_GP -> SRAM_A13
- U3 pad 14: RW -> VGG
- U3 pad 15: AD15 -> SRAM_A14
- U3 pad 16: AD14 -> SRAM_WE
- U3 pad 17: AD13 -> PV
- U3 pad 18: AD12 -> SRAM_CS
- U3 pad 19: AD11 -> PC1500_SENSE
- U3 pad 2: PC1500_SENSE -> AD11
- U3 pad 20: VGG -> DME0
- U3 pad 3: SRAM_CS -> AD12
- U3 pad 4: PV -> AD13
- U3 pad 5: SRAM_WE -> AD14
- U3 pad 6: SRAM_A14 -> AD15
- U3 pad 7: VGG -> RW
- U3 pad 8: SRAM_A13 -> SCL_GP
- U3 pad 9: unconnected-(U3-IO7-Pad9) -> SDA_GP
- U9 pad 1: TRIG_RD -> VCC
- U9 pad 10: GND -> TRIG_RD
- U9 pad 11: Net-(U9-IO6) -> GND
- U9 pad 12: SDA_GP_U9 -> TRIG_WR
- U9 pad 13: SCL_GP_U9 -> DME0
- U9 pad 14: RW -> VCC
- U9 pad 15: Net-(U9-IO4) -> OD
- U9 pad 16: AD14 -> unconnected-(U9-IO10-Pad16)
- U9 pad 18: OD -> unconnected-(U9-IO12-Pad18)
- U9 pad 19: DME0 -> GREENPAK2_IO13
- U9 pad 2: GREENPAK2_IO13 -> AD11
- U9 pad 20: VCC -> GREENPAK2_IO14
- U9 pad 3: AD15 -> AD12
- U9 pad 4: AD14 -> AD13
- U9 pad 5: AD13 -> AD14
- U9 pad 6: AD12 -> AD15
- U9 pad 7: +3V3 -> RW
- U9 pad 8: AD11 -> SCL_GP_U9
- U9 pad 9: TRIG_WR -> SDA_GP_U9
- X1 pad 2: XOUT -> GND
- X1 pad 3: (no net) -> XOUT
- X1 pad 4: (no net) -> GND
Routing:
- net (no net): track 0.00 -> 52.5 mm, vias 0 -> 1
- net Net-(U9-IO4): track 26.9 -> 0.00 mm, vias 2 -> 0
- net Net-(U9-IO6): track 25.6 -> 0.00 mm, vias 2 -> 0
- net SD_MOSI: track 23.3 -> 25.7 mm
- net VGG: track 11.1 -> 9.06 mm, vias 9 -> 7
- net DME0: track 24.3 -> 25.4 mm, vias 5 -> 6
- net SD_CS: track 26.1 -> 27.1 mm
- net RW: track 37.4 -> 38.4 mm, vias 3 -> 4
- net SRAM_A11: track 0.00 -> 0.47 mm, vias 0 -> 1
- net TRIG_RD: track 8.27 -> 8.69 mm, vias 2 -> 3
- net OD: vias 2 -> 4
